File: HDK/Power/AMS1117.kicad_sch (KiCad schematic)
At the start: 6 parts, among them U201 AMS1117-3.3, U202 AMS1117-5.0

Commit message: added content
Parts:
- added C101, C103, C105, C108: 100n, symbol scottcjx-common-parts:100nF
- added C102, C104, C106, C107: 10u, symbol scottcjx-common-parts:10uF
- added D101, D103: CESD5V0D3, symbol scottcjx-common-parts:CESD5V0
- added D102: CESD12VD3, symbol scottcjx-common-parts:CESD12V
- added D104: CESD3V3D3, symbol scottcjx-common-parts:CESD3V3
- added U101: AMS1117-3.3, Package_TO_SOT_SMD:SOT-223-3_TabPin2, symbol Regulator_Linear:AMS1117-3.3
- added U102: AMS1117-5.0, Package_TO_SOT_SMD:SOT-223-3_TabPin2, symbol Regulator_Linear:AMS1117-5.0
Connections:
- net +3V3: now also C103.1, C104.1, D104.1 (K), U101.2 (VO)
- net +5V: now also C101.1, C102.1, C107.1, C108.1, D101.1 (K), D103.1 (K), U101.3 (VI), U102.2 (VO)
- net GND: now also C101.2, C102.2, C103.2, C104.2, C105.2, C106.2, C107.2, C108.2, D101.2 (A), D102.2 (A), D103.2 (A), D104.2 (A), U101.1 (GND), U102.1 (GND)
- net VCC: now also C105.1, C106.1, D102.1 (K), U102.3 (VI)
Other:
- note added: "If 12V not used as V_{in}, use suitable TVS Diode"
- note added: "If 5V not used as V_{in}, use suitable TVS Diode"
- note added: "Recommended to use 5V as V_{in} here"
- note added: "V_{in}-min: 6.5v V_{in}-typ: 12v V_{in}-max: 15v"
